Commit message: Add bessica bringup launch

File: bessica_d_description/urdf/bessica_D_v2_1.urdf (robot description, URDF)
Before this commit: robot bessica_d_v2_1, 23 links, 22 joints
Joints:
- joint left_arm_gripper_joint2: mimic (none) -> joint=left_arm_gripper_joint1 multiplier=-1 offset=0
- joint left_arm_joint3: axis 0 0 -1 -> 0 0 1
- joint left_arm_joint5: axis 0 0 -1 -> 0 0 1
- joint right_arm_gripper_joint2: mimic (none) -> joint=right_arm_gripper_joint1 multiplier=-1 offset=0
- joint right_arm_joint1: axis 0 0 -1 -> 0 0 1
- joint right_arm_joint4: axis 0 0 -1 -> 0 0 1
- joint right_arm_joint6: axis 0 0 -1 -> 0 0 1
- joint right_arm_joint7: axis 0 0 -1 -> 0 0 1
